File: sandbox/radishes/sensor_interface_brd/sableye/sableye.sch (KiCad schematic (older format))
At the start: 8 parts, among them U2 ADS1115, U3 ADS1115, U4 ADS1115, U5 ADS1115

Commit message: some minor tweaks
Parts:
- added J? (x3): Conn_01x02_Female, symbol Connector:Conn_01x02_Female
- added J?: Conn_01x04_Female, symbol Connector:Conn_01x04_Female
- U2, U3, U4, U5: symbol devs:ADS1115 -> sableye-rescue:ADS1115-devs
Connections:
- wire segments 39 -> 46
Changed lines of the file:
@@
 $Descr A4 11693 8268
 encoding utf-8
-Sheet 2 3
+Sheet 1 1
 Title ""
 Date ""
@@
 $EndDescr
 $Comp
-L devs:ADS1115 U3
+L sableye-rescue:ADS1115-devs U3
 U 1 1 59B29154
 P 6250 1750
@@
 $EndComp
 $Comp
-L devs:ADS1115 U4
+L sableye-rescue:ADS1115-devs U4
 U 1 1 59B29192
 P 6250 3050
@@
 $EndComp
 $Comp
-L devs:ADS1115 U5
+L sableye-rescue:ADS1115-devs U5
 U 1 1 59B291B4
 P 6250 4350
@@
 $EndComp
 $Comp
-L devs:ADS1115 U2
+L sableye-rescue:ADS1115-devs U2
 U 1 1 59B29207
 P 6200 5650
@@
 	1    0    0    -1
 $EndComp
-Text HLabel 4400 1500 0    60   UnSpc ~ 0
-VDD
-Wire Wire Line
-	4600 2800 5800 2800
-Wire Wire Line
-	4600 4100 5800 4100
-Wire Wire Line
-	4600 5400 5750 5400
-Wire Wire Line
-	4400 1500 4600 1500
-Wire Wire Line
-	4600 1500 4600 2800
-Connection ~ 4600 1500
-Connection ~ 4600 2800
-Connection ~ 4600 4100
+Text HLabel 5700 1500 0    60   UnSpc ~ 0
+VDD
 $Comp
 L power:GND #PWR07
@@
 Wire Wire Line
 	5650 5700 5750 5700
-Wire Wire Line
-	4600 3200 5800 3200
 Text HLabel 5750 3300 0    60   Output ~ 0
 ALERT_0x49
@@
 	5300 1900 5300 1600
 Connection ~ 5300 1600
-Connection ~ 4600 3200
 Wire Wire Line
 	5750 5800 5700 5800
@@
 Connection ~ 5750 4400
 Wire Wire Line
-	4600 1500 5800 1500
-Wire Wire Line
-	4600 2800 4600 3200
-Wire Wire Line
-	4600 4100 4600 5400
-Wire Wire Line
 	5300 1600 5800 1600
-Wire Wire Line
-	4600 3200 4600 4100
 Wire Wire Line
 	5700 5600 5750 5600
@@
 	1    0    0    -1
 $EndComp
+$Comp
+L Connector:Conn_01x02_Female J?
+U 1 1 5E39DB78
+P 3500 1600
+F 0 "J?" H 3394 1275 50  0000 C CNN
+F 1 "Conn_01x02_Female" H 3394 1366 50  0000 C CNN
+F 2 "" H 3500 1600 50  0001 C CNN
+F 3 "~" H 3500 1600 50  0001 C CNN
+	1    3500 1600
+	-1   0    0    1
+$EndComp
+$Comp
+L Connector:Conn_01x02_Female J?
+U 1 1 5E39DCA3
+P 3550 4350
+F 0 "J?" H 3444 4025 50  0000 C CNN
+F 1 "Conn_01x02_Female" H 3444 4116 50  0000 C CNN
+F 2 "" H 3550 4350 50  0001 C CNN
+F 3 "~" H 3550 4350 50  0001 C CNN
+	1    3550 4350
+	-1   0    0    1
+$EndComp
+Text HLabel 3800 1500 2    60   UnSpc ~ 0
+VDD
+$Comp
+L power:GND #PWR?
+U 1 1 5E39DCFF
+P 3800 1600
+F 0 "#PWR?" H 3800 1350 50  0001 C CNN
+F 1 "GND" H 3800 1450 50  0000 C CNN
+F 2 "" H 3800 1600 50  0000 C CNN
+F 3 "" H 3800 1600 50  0000 C CNN
+	1    3800 1600
+	1    0    0    -1
+$EndComp
+Wire Wire Line
+	3800 1600 3700 1600
+Wire Wire Line
+	3700 1500 3800 1500
+Text HLabel 3850 4250 2    60   Input ~ 0
+SCLK
+Text HLabel 3850 4350 2    60   BiDi ~ 0
+SDA
+Wire Wire Line
+	3850 4250 3750 4250
+Wire Wire Line
+	3850 4350 3750 4350
+$Comp
+L Connector:Conn_01x04_Female J?
+U 1 1 5E3A01C2
+P 3500 2800
+F 0 "J?" H 3394 2375 50  0000 C CNN
+F 1 "Conn_01x04_Female" H 3394 2466 50  0000 C CNN
+F 2 "" H 3500 2800 50  0001 C CNN
+F 3 "~" H 3500 2800 50  0001 C CNN
+	1    3500 2800
+	-1   0    0    1
+$EndComp
+Text HLabel 3750 2900 2    60   Output ~ 0
+ALERT_0x48
+Text HLabel 3750 2800 2    60   Output ~ 0
+ALERT_0x49
+Text HLabel 3750 2700 2    60   Output ~ 0
+ALERT_0x4A
+Text HLabel 3750 2600 2    60   Output ~ 0
+ALERT_0x4B
+Wire Wire Line
+	3700 2600 3750 2600
+Wire Wire Line
+	3750 2700 3700 2700
+Wire Wire Line
+	3700 2800 3750 2800
+Wire Wire Line
+	3750 2900 3700 2900
+Wire Wire Line
+	5700 1500 5800 1500
+Text HLabel 5050 2800 0    60   UnSpc ~ 0
+VDD
+Wire Wire Line
+	5050 2800 5100 2800
+Wire Wire Line
+	5800 3200 5100 3200
+Wire Wire Line
+	5100 3200 5100 2800
+Connection ~ 5100 2800
+Wire Wire Line
+	5100 2800 5800 2800
+Text HLabel 5700 4100 0    60   UnSpc ~ 0
+VDD
+Wire Wire Line
+	5700 4100 5800 4100
+Text HLabel 5650 5400 0    60   UnSpc ~ 0
+VDD
+Wire Wire Line
+	5650 5400 5750 5400
+$Comp
+L Connector:Conn_01x02_Female J?
+U 1 1 5E3AACCE
+P 3500 2150
+F 0 "J?" H 3394 1825 50  0000 C CNN
+F 1 "Conn_01x02_Female" H 3394 1916 50  0000 C CNN
+F 2 "" H 3500 2150 50  0001 C CNN
+F 3 "~" H 3500 2150 50  0001 C CNN
+	1    3500 2150
+	-1   0    0    1
+$EndComp
+Text HLabel 3800 2050 2    60   Input ~ 0
+SCLK
+Text HLabel 3800 2150 2    60   BiDi ~ 0
+SDA
+Wire Wire Line
+	3800 2050 3700 2050
+Wire Wire Line
+	3800 2150 3700 2150
 $EndSCHEMATC
