File: sandbox/radishes/sensor_interface_brd/sableye/sableye.kicad_pcb (KiCad board)
At the start: 2 copper layers, 17 parts, among them P1 CONN_01X04, P2 CONN_01X04, P3 CONN_01X04, P4 CONN_01X04, U2 ADS1115, U3 ADS1115, U4 ADS1115, U5 ADS1115

Commit message: generated netlist, simplified
Parts:
- removed C1, C2: CP, Capacitors_THT:CP_Radial_D10.0mm_P5.00mm
- removed C3: 100pF, Capacitors_THT:C_Axial_L12.0mm_D6.5mm_P15.00mm_Horizontal
- removed D1, D3: D, Diodes_THT:D_DO-15_P12.70mm_Horizontal
- removed D2: LED, LEDs:LED_D5.0mm
- removed L1: L, Inductors_THT:L_Axial_L9.5mm_D4.0mm_P12.70mm_Horizontal_Fastron_SMCC
- removed P1, P2, P3, P4: CONN_01X04, Connectors_Terminal_Blocks:TerminalBlock_Pheonix_MPT-2.54mm_4pol
- removed R1: R, Resistors_THT:R_Axial_DIN0204_L3.6mm_D1.6mm_P5.08mm_Horizontal
- removed R2: 100, Resistors_THT:R_Axial_DIN0204_L3.6mm_D1.6mm_P5.08mm_Horizontal
- removed U2, U3, U4, U5: ADS1115, Connectors_Terminal_Blocks:TerminalBlock_Pheonix_MPT-2.54mm_10pol
